File: USB_DebugCable.brd (EAGLE design)
At the start: 36.6 x 11.6 mm, 28 parts, among them U1 FT232RQ, U2 TPS71701, U3 TPS71718

Commit message: Schematic, board and library updates
Signed-off-by: Daniel Ghilinta <ghilinta.daniel@gmail.com>
Parts:
- removed 3V3, GND, GND1, RXD, TXD: WIREPAD2,15/1,0, wirepad:2,15/1,0
- removed PTC1: 33 Ohm, rcl:R0603
- removed RX, TX: (no value), led:CHIPLED_0603
- removed U$2: (no value), untitled:LOGO_ANDROID_USB
- removed U$3: (no value), frames:DOCFIELD
- removed U1: FT232RQ, ftdichip:QFN32
- removed U2: TPS71701, TPS717xx:SC70-5
- removed U3: TPS71718, TPS717xx:SC70-5
- added C9: .1u, rcl-2:C0402K
- added IC1: FT232RLSSOP, SparkFun:SSOP28DB
- added IC2: APE8800N-33, linear:SOT23
- added IC3: MCP1700T-18, linear:SOT23
- added JP1: USB-A-H, SparkFun-Connectors:USB-A-H
- added JP2, JP3, JP4, JP5: (no value), adafruit:1X01
- added JP6: (no value), adafruit:1X06-CLEANBIG
- added LED1, LED2, LED3: (no value), adafruit:CHIPLED_0603
- added PF1: PTC-F0603MP, polyswitch:F0603MP
- added R6: 220R, rcl-2:R0603
- C1, C3: value .1uF -> 1u; device rcl:C0402 -> rcl-2:C0603K
- C2: value 4.7uF -> 1u; device rcl:C0402 -> rcl-2:C0603K
- C4: value 1uF -> 1u; device rcl:C0402 -> rcl-2:C0603K
- C5: value 1uF -> 10u; device rcl:C0402 -> rcl-2:C0603K
- C6: value .1uF -> 10u; device rcl:C0402 -> rcl-2:C0603K
- C7: value 1uF -> .1u; device rcl:C0402 -> rcl-2:C0603K
- C8: value 10nF -> .1u; device rcl:C0402 -> rcl-2:C0402K
- FB1: value 33 -> (none); device rcl:C0402 -> m-pad-2.1:0603
- R1: value 120 -> 1k; device rcl:R0402 -> rcl-2:R0603
- R2: value 120 -> 120R; device rcl:R0402 -> rcl-2:R0603
- R3: value 33 -> 120R; device rcl:R0402 -> rcl-2:R0603
- R4: value 976K -> 33R; device rcl:R0402 -> rcl-2:R0603
- R5: value 301K -> 33R; device rcl:R0402 -> rcl-2:R0603
- U$1: value USB_A_PLUG -> JACK3.5_4; device USB_DEBUG:MOLEX_48037-1000 -> jack_35_4:3.5MM4
- moved U$1 48.3 mm to (49.9, 16.3), turned to 180 degrees
- moved R2 27.5 mm to (38.7, 19.1)
- moved C7 24.4 mm to (48.0, 20.1), turned to 0 degrees
- moved C8 21.1 mm to (25.7, 13.7), turned to 270 degrees
- moved C5 15.3 mm to (8.89, 10.9), turned to 90 degrees
- moved R3 14.5 mm to (38.7, 21.2), turned to 0 degrees
- moved R5 11.8 mm to (37.6, 4.45), turned to 270 degrees
- moved R4 10.7 mm to (37.8, 9.91)
- moved C6 10.2 mm to (10.7, 12.3), turned to 90 degrees
- moved C1 9.82 mm to (18.0, 11.9), turned to 270 degrees
- moved R1 9.75 mm to (24.9, 9.53), turned to 270 degrees
- moved C4 9.05 mm to (12.2, 10.5)
- moved C3 7.85 mm to (21.2, 8.38), turned to 180 degrees
- moved C2 7.49 mm to (15.0, 8.51), turned to 180 degrees
- moved FB1 5.24 mm to (7.37, 7.87), turned to 270 degrees
Connections:
- removed net MIC_PIN_PROTECTED: 3V3.1, PTC1.2
- removed net RXD: RXD.1, U1.2
- removed net RXLED: R2.1, U1.21
- removed net TXD: R3.2, TXD.1
- removed net TXD_UNFILTERED: R3.1, U1.30
- removed net TXLED: R1.1, U1.22
- removed net USB_D+: U$1.USB_D+, U1.14
- removed net USB_D-: U$1.USB_D-, U1.15
- removed net VBUS_UNFILTERED: C8.1, FB1.1, U$1.VDD
- removed net VCC: C2.1, C5.1, C6.1, FB1.2, U1.19, U2.EN, U2.IN, U3.EN, U3.IN
- removed net VDD_1V8: C4.1, U1.1, U3.OUT
- removed net VDD_3V3: C1.1, C3.1, RX.A, TX.A, U1.16
- removed net VDD_3V36: C7.1, PTC1.1, R4.2, U2.OUT
- new net 1V8: C3.1, IC3.2, JP4.1, JP6.3
- new net 3V3: C2.1, C7.1, IC2.2, JP3.1, JP6.2, LED1.A, LED2.A, R5.1
- new net 3V3OUT: C9.1, IC1.17
- new net 5V: C1.1, C4.1, C5.1, C6.1, C8.1, IC1.20, IC2.3, IC3.3, JP2.1, JP6.1, LED3.A, PF1.2
- new net D+: IC1.15, JP1.D+
- new net D-: IC1.16, JP1.D-
- new net N$4: FB1.2, PF1.1
- new net N$5: IC1.23, R2.1
- new net N$6: IC1.22, R3.1
- new net N$7: LED1.C, R2.2
- new net N$8: LED2.C, R3.2
- new net N$9: LED3.C, R6.2
- new net RX: IC1.5, JP6.5, U$1.RX_1, U$1.RX_2
- new net TX: JP6.4, R4.1, U$1.TX
- new net VCCIO: IC1.4, JP5.1, R1.2
- net GND: now also C9.2, IC1.18, IC1.21, IC1.25, IC1.26, IC1.7, IC2.1, IC3.1, JP1.GND, JP6.6, R1.1, R6.1; no longer GND.1, GND1.1, R5.1, U$1.SHIELD1, U$1.SHIELD2, U1.17, U1.20, U1.24, U1.26, U1.4, U2.GND, U3.GND
- net N$1: now also FB1.1, JP1.VBUS; no longer R4.1, R5.2, U2.FB
- net N$2: now also R5.2, U$1.MIC_1, U$1.MIC_2; no longer R1.2, TX.C
- net N$3: now also IC1.1, R4.2; no longer R2.2, RX.C
Routing:
- net GND: track 99.4 -> 18.6 mm, vias 7 -> 29
- net 5V: track 0.00 -> 78.7 mm
- net 3V3: track 0.00 -> 72.4 mm, vias 0 -> 3
- net 1V8: track 0.00 -> 47.4 mm
- net VCC: track 30.5 -> 0.00 mm, vias 2 -> 0
- net D-: track 0.00 -> 25.7 mm
- net D+: track 0.00 -> 25.1 mm
- net VDD_3V3: track 24.4 -> 0.00 mm, vias 3 -> 0
- net RXD: track 21.0 -> 0.00 mm
- net RX: track 0.00 -> 20.3 mm
- net N$6: track 0.00 -> 16.4 mm
- net TXD_UNFILTERED: track 15.5 -> 0.00 mm, vias 2 -> 0
- net VCCIO: track 0.00 -> 15.2 mm
- net TX: track 0.00 -> 15.2 mm
- net N$5: track 0.00 -> 14.6 mm
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Other:
- board size 36.6 x 11.6 mm -> 55.5 x 25.7 mm
- board text removed: "(C) 2012, Google Inc."
- board text removed: "(C) Google Inc. 2012"
- board text removed: "1. Solder Mask - RED"
- board text removed: "11.6mm"
- board text removed: "2"
- board text removed: "2. 1oz Copper after plating"
- board text removed: "3. Board thickness 62mils nominal."
- board text removed: "36.6mm"
- board text removed: "4. Silkscreen - WHITE"
- board text removed: "5. Materials are to be ROHS and UL 94VO compliant"
- board text removed: "6. Surface finish is to be ENIG"
- board text removed: "7. Fabricate to IPC-600 Class 2 spec"
- board text removed: "Fab Notes:"
