File: USB_DebugCable.sch (EAGLE design)
At the start: 26 parts, among them U1 FT232RQ, U2 TPS71701, U3 TPS71718

Commit message: Schematic, board and library updates
Signed-off-by: Daniel Ghilinta <ghilinta.daniel@gmail.com>
Parts:
- removed 3V3, GND, GND1, RXD, TXD: WIREPAD2,15/1,0, wirepad:WIREPAD2,15/1,0
- removed PTC1: 33 Ohm, rcl:R-US_R0603
- removed RX, TX: (no value), led:LEDCHIPLED_0603
- removed U1: FT232RQ, ftdichip:FT232RQ
- removed U2: TPS71701, TPS717xx:TPS717XX
- removed U3: TPS71718, TPS717xx:TPS717XX
- added C9: .1u, rcl-2:C-EUC0402K
- added IC1: FT232RLSSOP, SparkFun:FT232RLSSOP
- added IC2: APE8800N-33, linear:MCP1703CB
- added IC3: MCP1700T-18, linear:MCP1703CB
- added JP1: USB-A-H, SparkFun-Connectors:USB-A-H
- added JP2, JP3, JP4, JP5: (no value), adafruit:PINHD-1X1
- added JP6: (no value), adafruit:PINHD-1X6CB
- added LED1, LED2, LED3: (no value), adafruit:LEDCHIPLED_0603
- added PF1: PTC-F0603MP, polyswitch:PTC-F0603MP
- added R6: 220R, rcl-2:R-EU_R0603
- C1, C3: value .1uF -> 1u; device rcl:C-USC0402 -> rcl-2:C-EUC0603K
- C2: value 4.7uF -> 1u; device rcl:C-USC0402 -> rcl-2:C-EUC0603K
- C4: value 1uF -> 1u; device rcl:C-USC0402 -> rcl-2:C-EUC0603K
- C5: value 1uF -> 10u; device rcl:C-USC0402 -> rcl-2:C-EUC0603K
- C6: value .1uF -> 10u; device rcl:C-USC0402 -> rcl-2:C-EUC0603K
- C7: value 1uF -> .1u; device rcl:C-USC0402 -> rcl-2:C-EUC0603K
- C8: value 10nF -> .1u; device rcl:C-USC0402 -> rcl-2:C-EUC0402K
- FB1: value 33 -> (none); device rcl:C-USC0402 -> m-pad-2.1:FERRITE-BEADA
- R1: value 120 -> 1k; device rcl:R-US_R0402 -> rcl-2:R-EU_R0603
- R2: value 120 -> 120R; device rcl:R-US_R0402 -> rcl-2:R-EU_R0603
- R3: value 33 -> 120R; device rcl:R-US_R0402 -> rcl-2:R-EU_R0603
- R4: value 976K -> 33R; device rcl:R-US_R0402 -> rcl-2:R-EU_R0603
- R5: value 301K -> 33R; device rcl:R-US_R0402 -> rcl-2:R-EU_R0603
- U$1: value USB_A_PLUG -> JACK3.5_4; device USB_DEBUG:USB_A_PLUG -> jack_35_4:JACK3.5_4
Connections:
- removed net MIC_PIN_PROTECTED: 3V3.P, PTC1.2
- removed net RXD: RXD.P, U1.RXD
- removed net RXLED: R2.1, U1.CBUS1
- removed net TXD: R3.2, TXD.P
- removed net TXD_UNFILTERED: R3.1, U1.TXD
- removed net TXLED: R1.1, U1.CBUS0
- removed net USB_D+: U$1.USB_D+, U1.USBDP
- removed net USB_D-: U$1.USB_D-, U1.USBDM
- removed net VBUS_UNFILTERED: C8.1, FB1.1, U$1.VBUS
- removed net VCC: C2.1, C5.1, C6.1, FB1.2, U1.VCC, U2.EN, U2.IN, U3.EN, U3.IN
- removed net VDD_1V8: C4.1, U1.VCCIO, U3.OUT
- removed net VDD_3V3: C1.1, C3.1, RX.A, TX.A, U1.3V3OUT
- removed net VDD_3V36: C7.1, PTC1.1, R4.2, U2.OUT
- new net 1V8: C3.1, IC3.VO, JP4.1, JP6.3
- new net 3V3: C2.1, C7.1, IC2.VO, JP3.1, JP6.2, LED1.A, LED2.A, R5.1
- new net 3V3OUT: C9.1, IC1.3V3OUT
- new net 5V: C1.1, C4.1, C5.1, C6.1, C8.1, IC1.VCC, IC2.VI, IC3.VI, JP2.1, JP6.1, LED3.A, PF1.2
- new net D+: IC1.USBDP, JP1.D-
- new net D-: IC1.USBDM, JP1.D+
- new net N$4: FB1.2, PF1.1
- new net N$5: IC1.TXLED, R2.1
- new net N$6: IC1.RXLED, R3.1
- new net N$7: LED1.C, R2.2
- new net N$8: LED2.C, R3.2
- new net N$9: LED3.C, R6.2
- new net RX: IC1.RXD, JP6.5, U$1.RX
- new net TX: JP6.4, R4.1, U$1.TX
- new net VCCIO: IC1.VCCIO, JP5.1, R1.2
- net GND: now also C9.2, IC1.AGND, IC1.GND18, IC1.GND21, IC1.GND7, IC1.TEST, IC2.GND, IC3.GND, JP1.VBUS, JP6.6, R1.1, R6.1; no longer GND.P, GND1.P, R5.1, U$1.SHLD1, U$1.SHLD2, U1.GND, U1.GND@1, U1.GND@2, U1.GND@A, U1.TEST, U2.GND, U3.GND
- net N$1: now also FB1.1, JP1.GND; no longer R4.1, R5.2, U2.FB
- net N$2: now also R5.2, U$1.MIC; no longer R1.2, TX.C
- net N$3: now also IC1.TXD, R4.2; no longer R2.2, RX.C
Other:
- note removed: "1% Tolerance"
- note removed: "A"
- note removed: "Blue LED (Part: LB Q39G-L2N2-35-1)"
- note removed: "Copyright 2012, 2014, Google Inc."
- note removed: "Input / L Audio"
- note removed: "No Warranty expressed or implied."
- note removed: "Output / R Audio"
- note removed: "RX_in"
- note removed: "TBA"
- note removed: "TX_out"
- note removed: "To MIC pin"
- note removed: "Wirepad 1.0mm diameter"
- note removed: "gnd"
- note removed: "mic"
- moved on the sheet: C1, C2, C3, C4, C5, C6, C7, C8
